File: OpenEVSE_PLUS_v6.5.1_KiCad/OpenEVSE_PLUS_v6.5.1.kicad_pcb (KiCad board)
At the start: 2 copper layers, 91.1 x 51.3 mm, 117 parts, among them IC1 LMV358, IC2 ATMEGA328P-AU, IC3 LM358, IC4 TC1044S, IC7 AQH2223, IC8 HCPL-2731S, M1 MOV, M2 MOV, M3 MOV, M4 MOV, Q1 16000, Q2 2222A, Q3 2222A, U1 AP63203

Commit message: Link the KiCad board to its schematic
Update PCB from Schematic (KiCad 10 GUI): re-link by reference, replace
footprints, update fields; 0 errors, 4 warnings (FID1-4 copper pad with
no symbol pin, no net in EAGLE either).

pcb_geomdiff.py (new) compared the board before and after with nets
matched by their pads: 686 segments, 63 vias, 6 zones, 21 graphics and
all 117 footprint placements/pads identical. Only the expected changes:
30 N$ nets renamed to Net-(...), 21 symbol fields copied, 3 connector
values filled, 5 open pads given unconnected-* nets, sheet paths added.

netcmp: 0 differing nets vs EAGLE .brd and vs the schematic netlist.
DRC unchanged (0 unconnected, 3 pre-existing errors). kicad-cli's
--schematic-parity names multi-unit nets differently from the GUI and
the netlist exporter (22 name-only conflicts); noted in the README.
Parts:
- I2C0: value (none) -> M04JST-PTH-VERT
- JP2: value (none) -> M06POLAR_LOCK
- PILOT0: value (none) -> M025MM
Connections:
- D1 pad 3: (no net) -> unconnected-(D1-AA-Pad3)
- D11 pad 3: (no net) -> unconnected-(D11-AA-Pad3)
- IC4 pad 6: (no net) -> unconnected-(IC4-LV-Pad6)
- IC4 pad 7: (no net) -> unconnected-(IC4-OSC-Pad7)
- IC7 pad P$5: (no net) -> unconnected-(IC7-5-PadP$5)
